File: Interface.kicad_sch (KiCad schematic)
At the start: 0 parts

Commit message: added a comment to the interface about constrains
Other:
- note added: "For transmitting the data, a well defined highly isolated interface is needed. The reason for the isolated interface is the fact, that this measurement device should be able to be operated at a high voltage supply. For this the isolation distance of 6kV is assumed. For class B2, this results in 30mm, which is also assumed to be on the very safe side for using on this PCB."
Changed lines of the file:
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@@
 (kicad_sch (version 20211123) (generator eeschema)
   (paper "A4")
+  (text "For transmitting the data, a well defined highly isolated interface is needed.\nThe reason for the isolated interface is the fact, that this measurement device\nshould be able to be operated at a high voltage supply. \nFor this the isolation distance of 6kV is assumed. For class B2, this results \nin 30mm, which is also assumed to be on the very safe side for using on this \nPCB."
+    (at 179.07 161.29 0)
+    (effects (font (size 1.6 1.6)) (justify left bottom))
+  )
 )
