File: InterfacePCside.kicad_sch (KiCad schematic)
At the start: 0 parts

Commit message: changed title block to meaningful information
Other:
- title: (none) -> Open Nano Amp Meter
Changed lines of the file:
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@@
 (kicad_sch (version 20211123) (generator eeschema)
   (paper "A4")
+  (title_block
+    (title "Open Nano Amp Meter")
+    (date "2022-11-17")
+    (rev "0.9")
+  )
 )
