File: CurrentMeasurement.kicad_sch (KiCad schematic)
At the start: 24 parts, among them U1 DDC112U, U5 REF3040

Commit message: added buffer to ref voltage generation
Parts:
- added C29: 10u, Capacitor_SMD:CP_Elec_4x3.9, symbol Device:C_Polarized
- added C30, C31: 100n, Capacitor_SMD:C_0603_1608Metric, symbol Device:C
- added R24: R, Resistor_SMD:R_0603_1608Metric, symbol Device:R
- added U14: OPA340UA, Package_SO:SOIC-8_3.9x4.9mm_P1.27mm, symbol Amplifier_Operational:OPA340UA
Connections:
- net +5VA: now also C31.1, U14.7 (V+)
- net GNDA: now also C29.2, C30.2, C31.2, U14.4 (V-)
- net VREF: now also C29.1, C30.1, R24.2
- net at C5.1, C6.1, R8.2: now also U14.3 (+)
- new net: R24.1, U14.2 (-), U14.6
